Commit message: 힘 센서 적용

File: src/robotarm_polishing/M0609/doosan-robot2/urdf/m0609_isaac_sim.urdf (robot description, URDF)
Before this commit: robot m0609, 9 links, 8 joints
Links:
- added link pad_tip
Joints:
- added joint link_6-pad_tip: type fixed, parent link_6, child pad_tip, origin xyz=0 0 0.085 rpy=0 0 0
